Commit message: changed

File: urdf/qs_bot.xacro (robot description, xacro)
@@ -68,5 +68,5 @@
       <origin rpy="0 0 0" xyz="-0.2476 -0.2193 -0.12"/>
       <geometry>
-        <mesh filename="package://qs_bot/meshes/base_frame.STL" scale="0.001 0.001 0.001"/>
+        <mesh filename="package://qsbot_simulation/meshes/base_frame.STL" scale="0.001 0.001 0.001"/>
         <!-- <box size="0.48 0.48 0.225"/> -->
       </geometry>
@@ -75,5 +75,5 @@
       <origin rpy="0 0 0" xyz="0 0 0"/>
       <geometry>
-        <!-- <mesh filename="package://qs_bot/meshes/base_frame.STL" scale="0.001 0.001 0.001"/> -->
+        <!-- <mesh filename="package://qsbot_simulation/meshes/base_frame.STL" scale="0.001 0.001 0.001"/> -->
         <box size="0.48 0.48 0.225"/>
       </geometry>
@@ -89,5 +89,5 @@
         <origin rpy= "${PI/2} 0 0" xyz= "${joint_wheel_match}"/>
         <geometry>
-          <mesh filename="package://qs_bot/meshes/mecanum_wheel.STL" scale="0.001 0.001 0.001"/>
+          <mesh filename="package://qsbot_simulation/meshes/mecanum_wheel.STL" scale="0.001 0.001 0.001"/>
         </geometry>
         <material name= "black"/>
@@ -96,5 +96,5 @@
         <origin rpy= "${PI/2} 0 0" xyz= "${joint_wheel_match}"/>
         <geometry>
-          <mesh filename="package://qs_bot/meshes/mecanum_wheel.STL" scale="0.001 0.001 0.001"/>
+          <mesh filename="package://qsbot_simulation/meshes/mecanum_wheel.STL" scale="0.001 0.001 0.001"/>
         </geometry>
       </collision>
@@ -136,5 +136,5 @@
       <!-- <origin rpy="0 0 0" xyz="-0.0375 0.0375 -0.01"/> -->
       <geometry>
-        <!--mesh filename="package://qs_bot/meshes/LiDAR.STL" scale="0.001 0.001 0.001"/-->
+        <!--mesh filename="package://qsbot_simulation/meshes/LiDAR.STL" scale="0.001 0.001 0.001"/-->
         <cylinder radius="0.05" length="0.04"/>
       </geometry>
